Commit message: Update inertial properties for Pelvis and Tibia links
Adjustment of inertia, so that the robot does not fall immediately after turning on

File: pepper_robot_description/urdf/pepper_legs.xacro (robot description, xacro)
@@ -25,11 +25,10 @@
 	</joint>
 	<link name="Pelvis">
-		<inertial>
-			<mass value="2.45917" />
-			<inertia ixx="0.034351" ixy="0" ixz="0.000223034" iyy="0.0303122" iyz="-8.37542e-05"
-				izz="0.0143771" />
-			<origin rpy="0 0 0" xyz="0.00237 0 -0.09654" />
-		</inertial>
-		<xacro:insert_visu_Pelvis />
+    <inertial>
+        <mass value="2.45917" />
+        <inertia ixx="0.04" ixy="0" ixz="0.0002" iyy="0.04" iyz="0" izz="0.02" />
+        <origin rpy="0 0 0" xyz="0.00237 0 -0.09654" />
+    </inertial>
+    <xacro:insert_visu_Pelvis />
 	</link>
 	<joint name="KneePitch" type="revolute">
@@ -41,11 +40,8 @@
 	</joint>
 	<link name="Tibia">
-		<inertial>
-			<mass value="11.6015" />
-			<inertia ixx="0.129229" ixy="-0.000401943" ixz="0.00048556" iyy="0.122839"
-				iyz="-1.01666e-08" izz="0.108168" />
-			<origin rpy="0 0 0" xyz="0.00220451 0 -0.185729" />
-		</inertial>
-		<xacro:insert_visu_Tibia />
+    <inertial>
+        <mass value="15.0" /> <inertia ixx="0.2" ixy="0" ixz="0" iyy="0.2" iyz="0" izz="0.15" />
+        <origin rpy="0 0 0" xyz="0 0 -0.2" /> </inertial>
+    <xacro:insert_visu_Tibia />
 	</link>
 	<joint name="base_footprint_joint" type="fixed">

Commit message: Update inertial properties for Pelvis and Tibia links
Added gazebo parameters for Tibia joint.

File: pepper_robot_description/urdf/pepper_legs.xacro (robot description, xacro)
@@ -49,9 +49,17 @@
 		<xacro:insert_visu_Tibia />
 	</link>
-	<joint name="base_footprint_joint" type="fixed">
-		<parent link="Tibia" />
-		<child link="base_footprint" />
-		<origin rpy="0 0 0" xyz="0 0 -0.334" />
-	</joint>
-	<link name="base_footprint" />
+    <joint name="base_footprint_joint" type="fixed">
+        <parent link="Tibia" />
+        <child link="base_footprint" />
+        <origin rpy="0 0 0" xyz="0 0 -0.334" />
+    </joint>
+    <link name="base_footprint" />
+    <gazebo reference="Tibia">
+        <mu1>1.5</mu1>
+        <mu2>1.5</mu2>
+        <kp>1000000.0</kp>
+        <kd>100.0</kd>
+        <minDepth>0.005</minDepth>
+        <maxVel>0.1</maxVel>
+    </gazebo>
 </robot>

Commit message: Update inertial properties for Pelvis and Tibia links

File: pepper_robot_description/urdf/pepper_legs.xacro (robot description, xacro)
@@ -25,12 +25,11 @@
 	</joint>
 	<link name="Pelvis">
-		<inertial>
-			<mass value="2.45917" />
-			<inertia ixx="0.034351" ixy="0" ixz="0.000223034" iyy="0.0303122" iyz="-8.37542e-05"
-				izz="0.0143771" />
-			<origin rpy="0 0 0" xyz="0.00237 0 -0.09654" />
-		</inertial>
-		<xacro:insert_visu_Pelvis />
-	</link>
+    <inertial>
+        <mass value="2.45917" />
+        <inertia ixx="0.04" ixy="0" ixz="0.0002" iyy="0.04" iyz="0" izz="0.02" />
+        <origin rpy="0 0 0" xyz="0.00237 0 -0.09654" />
+    </inertial>
+    <xacro:insert_visu_Pelvis />
+</link>
 	<joint name="KneePitch" type="revolute">
 		<parent link="Pelvis" />
@@ -41,17 +40,22 @@
 	</joint>
 	<link name="Tibia">
-		<inertial>
-			<mass value="11.6015" />
-			<inertia ixx="0.129229" ixy="-0.000401943" ixz="0.00048556" iyy="0.122839"
-				iyz="-1.01666e-08" izz="0.108168" />
-			<origin rpy="0 0 0" xyz="0.00220451 0 -0.185729" />
-		</inertial>
-		<xacro:insert_visu_Tibia />
-	</link>
-	<joint name="base_footprint_joint" type="fixed">
-		<parent link="Tibia" />
-		<child link="base_footprint" />
-		<origin rpy="0 0 0" xyz="0 0 -0.334" />
-	</joint>
-	<link name="base_footprint" />
+    <inertial>
+        <mass value="15.0" /> <inertia ixx="0.2" ixy="0" ixz="0" iyy="0.2" iyz="0" izz="0.15" />
+        <origin rpy="0 0 0" xyz="0 0 -0.2" /> </inertial>
+    <xacro:insert_visu_Tibia />
+</link>
+	 <joint name="base_footprint_joint" type="fixed">
+        <parent link="Tibia" />
+        <child link="base_footprint" />
+        <origin rpy="0 0 0" xyz="0 0 -0.334" />
+    </joint>
+    <link name="base_footprint" />
+    <gazebo reference="Tibia">
+        <mu1>1.5</mu1>
+        <mu2>1.5</mu2>
+        <kp>1000000.0</kp>
+        <kd>100.0</kd>
+        <minDepth>0.005</minDepth>
+        <maxVel>0.1</maxVel>
+    </gazebo>
 </robot>
